File: rapid_tank_level_indicator_hardware/rapid_tank_level_indicator.kicad_pcb (KiCad board)
At the start: 2 copper layers, 50 x 643 mm, 87 parts, among them J1 Conn_01x04_Pin, J17 TC2050, J2 Conn_02x04_Top_Bottom, J3 Conn_02x04_Top_Bottom, SW1 KMR721NGLFS, SW2 KMR721NGLFS, U1 L7805, U10 MCP9700Ax-ETT, U11 TPD4E1U06, U12 MCP9700Ax-ETT, U13 MCP9700Ax-ETT, U14 MCP9700Ax-ETT, U15 MCP9700Ax-ETT, U16 MCP2562-E-SN, U2 L7805, U3 STM32F105RCTx, U4 MCP9700Ax-ETT, U5 AZ1117-3.3, U6 MCP9700Ax-ETT, U7 MCP9700Ax-ETT, U8 MCP9700Ax-ETT, U9 MCP9700Ax-ETT, Y1 8MHz 12pF

Commit message: add connector and rc-filter
Parts:
- removed D1, D10, D11, D12, D13, D14, D15, D6, D8, D9: red, LED_SMD:LED_0603_1608Metric
- removed R26, R30, R32: 1k, Resistor_SMD:R_0402_1005Metric
- removed U2: L7805, Package_TO_SOT_SMD:TO-252-2
- added C18: 1u, Capacitor_SMD:C_0402_1005Metric, F.Cu at (139.5, 56.7)
- added C19: 1u, Capacitor_SMD:C_0402_1005Metric, F.Cu at (137.6, 56.2)
- added C22: 1u, Capacitor_SMD:C_0402_1005Metric, F.Cu at (138.6, 53.8)
- added C23: 1u, Capacitor_SMD:C_0402_1005Metric, F.Cu at (150.5, 55.8)
- added C26: 1u, Capacitor_SMD:C_0402_1005Metric, F.Cu at (148.6, 56.1)
- added C27: 1u, Capacitor_SMD:C_0402_1005Metric, F.Cu at (144.9, 56.3)
- added C28: 1u, Capacitor_SMD:C_0402_1005Metric, F.Cu at (146.7, 56.6)
- added C30: 1u, Capacitor_SMD:C_0402_1005Metric, F.Cu at (136.6, 53.6)
- added J4: Conn_01x12, custom_parts_lib:FFC3B07_pad, B.Cu at (136.0, 71.5)
- added J5: FFC3B07-12-T, custom_parts_lib:FFC3B0712T, F.Cu at (136.1, 63.0)
- added R12: 1k, Resistor_SMD:R_0402_1005Metric, F.Cu at (158.0, 48.2)
- added R13: 10k, Resistor_SMD:R_0402_1005Metric, F.Cu at (145.3, 57.7)
- added R14: 10k, Resistor_SMD:R_0402_1005Metric, F.Cu at (146.3, 58.1)
- added R15: 10k, Resistor_SMD:R_0402_1005Metric, F.Cu at (136.6, 54.6)
- added TP1: TestPoint, TestPoint:TestPoint_Pad_D1.0mm, F.Cu at (138.2, 649.3)
- added TP10: TestPoint, TestPoint:TestPoint_Pad_D1.0mm, F.Cu at (135.0, 126.8)
- added TP2: TestPoint, TestPoint:TestPoint_Pad_D1.0mm, F.Cu at (135.0, 360.2)
- added TP3: TestPoint, TestPoint:TestPoint_Pad_D1.0mm, F.Cu at (135.0, 593.9)
- added TP4: TestPoint, TestPoint:TestPoint_Pad_D1.0mm, F.Cu at (135.0, 301.8)
- added TP5: TestPoint, TestPoint:TestPoint_Pad_D1.0mm, F.Cu at (135.0, 535.1)
- added TP6: TestPoint, TestPoint:TestPoint_Pad_D1.0mm, F.Cu at (135.0, 243.4)
- added TP7: TestPoint, TestPoint:TestPoint_Pad_D1.0mm, F.Cu at (135.0, 476.9)
- added TP8: TestPoint, TestPoint:TestPoint_Pad_D1.0mm, F.Cu at (134.9, 185.3)
- added TP9: TestPoint, TestPoint:TestPoint_Pad_D1.0mm, F.Cu at (135.0, 418.5)
- C13: value 330n -> 1u; footprint Capacitor_SMD:C_0603_1608Metric -> Capacitor_SMD:C_0402_1005Metric
- C14: value 100n -> 1u
- D4: value RB070MM-30TR -> red; footprint Diode_SMD:D_SOD-123F -> LED_SMD:LED_0603_1608Metric
- R1: value 220 -> 1k5
- R10, R11, R4, R5, R6, R7, R9: value 1k -> 10k
- R3: value 220 -> 1k
- moved R4 415.3 mm to (141.4, 58.3), turned to 180 degrees
- moved R5 357.5 mm to (139.5, 57.7), turned to 180 degrees
- moved R6 299.1 mm to (142.9, 57.8)
- moved R7 241.3 mm to (137.6, 57.1), turned to 180 degrees
- moved R9 185.6 mm to (138.6, 54.8), turned to 180 degrees
- moved R10 124.9 mm to (148.2, 57.8)
- moved R11 68.5 mm to (150.0, 57.2)
- moved R3 33.3 mm to (158.0, 49.8), turned to 180 degrees
- moved D4 31.1 mm to (155.6, 49.8), turned to 0 degrees
- moved D5 28.9 mm to (155.6, 48.2), turned to 0 degrees
- moved C14 21.6 mm to (141.3, 57.3)
- moved C13 21.4 mm to (143.0, 56.3)
- moved C12 7.15 mm to (124.8, 42.9)
- moved D2 7.15 mm to (124.8, 45.8)
- moved D3 7.15 mm to (126.8, 47.3)
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Connections:
- C13 pad 1: GND -> Net-(U3-PA7)
- C13 pad 2: main_voltage -> GND
- C14 pad 1: GND -> Net-(U3-PA6)
- C14 pad 2: Net-(D4-A) -> GND
- D4 pad 1: +5V -> STAT_LED1
- D5 pad 1: GND -> STAT_LED2
- R10 pad 1: +3.3V -> Net-(U3-PB0)
- R10 pad 2: Net-(D14-A) -> TEMP_2_con
- R11 pad 1: +3.3V -> Net-(U3-PB1)
- R11 pad 2: Net-(D15-A) -> TEMP_1_con
- R3 pad 1: Net-(D4-A) -> +3.3V
- R3 pad 2: Net-(D5-A) -> Net-(D4-A)
- R4 pad 1: +3.3V -> Net-(U3-PA6)
- R4 pad 2: Net-(D8-A) -> TEMP_6_con
- R5 pad 1: +3.3V -> Net-(U3-PA5)
- R5 pad 2: Net-(D10-A) -> TEMP_7_con
- R6 pad 1: +3.3V -> Net-(U3-PA7)
- R6 pad 2: Net-(D11-A) -> TEMP_5_con
- R7 pad 1: +3.3V -> Net-(U3-PA4)
- R7 pad 2: Net-(D12-A) -> TEMP_8_con
- R9 pad 1: +3.3V -> Net-(U3-PA3)
- R9 pad 2: Net-(D13-A) -> TEMP_9_con
- U10 pad 1: +5V -> +5V_post_con
- U10 pad 3: GND -> GND_pos_con
- U12 pad 1: +5V -> +5V_post_con
- U12 pad 3: GND -> GND_pos_con
- U13 pad 1: +5V -> +5V_post_con
- U13 pad 3: GND -> GND_pos_con
- U14 pad 1: +5V -> +5V_post_con
- U14 pad 3: GND -> GND_pos_con
- U15 pad 1: +5V -> +5V_post_con
- U15 pad 3: GND -> GND_pos_con
- U3 pad 10: STAT_LED7 -> unconnected-(U3-PC2-Pad10)
- U3 pad 11: STAT_LED8 -> unconnected-(U3-PC3-Pad11)
- U3 pad 17: TEMP_9 -> Net-(U3-PA3)
- U3 pad 20: TEMP_8 -> Net-(U3-PA4)
- U3 pad 21: TEMP_7 -> Net-(U3-PA5)
- U3 pad 22: TEMP_6 -> Net-(U3-PA6)
- U3 pad 23: TEMP_5 -> Net-(U3-PA7)
- U3 pad 24: TEMP_4 -> Net-(U3-PC4)
- U3 pad 25: TEMP_3 -> Net-(U3-PC5)
- U3 pad 26: TEMP_2 -> Net-(U3-PB0)
- U3 pad 27: TEMP_1 -> Net-(U3-PB1)
- U3 pad 28: STAT_LED6 -> unconnected-(U3-PB2-Pad28)
- U3 pad 29: STAT_LED5 -> unconnected-(U3-PB10-Pad29)
- U3 pad 30: STAT_LED4 -> unconnected-(U3-PB11-Pad30)
- U3 pad 33: STAT_LED3 -> unconnected-(U3-PB12-Pad33)
- U3 pad 34: STAT_LED2 -> unconnected-(U3-PB13-Pad34)
- U3 pad 35: STAT_LED1 -> unconnected-(U3-PB14-Pad35)
- U3 pad 39: unconnected-(U3-PC8-Pad39) -> STAT_LED1
- U3 pad 40: unconnected-(U3-PC9-Pad40) -> STAT_LED2
- U3 pad 8: TEMP_10 -> Net-(U3-PC0)
- U4 pad 1: +5V -> +5V_post_con
- U4 pad 3: GND -> GND_pos_con
- U6 pad 1: +5V -> +5V_post_con
- U6 pad 3: GND -> GND_pos_con
- U7 pad 1: +5V -> +5V_post_con
- U7 pad 3: GND -> GND_pos_con
- U8 pad 1: +5V -> +5V_post_con
- U8 pad 3: GND -> GND_pos_con
- U9 pad 1: +5V -> +5V_post_con
- U9 pad 3: GND -> GND_pos_con
Routing:
- net +5V: track 766.4 -> 133.0 mm, vias 9 -> 8
- net +5V_post_con: track 0.00 -> 619.4 mm
- net STAT_LED1: track 610.6 -> 5.96 mm, vias 2 -> 0
- net +3.3V: track 790.9 -> 188.5 mm
- net STAT_LED2: track 551.6 -> 5.49 mm, vias 2 -> 0
- net STAT_LED3: track 492.1 -> 0.00 mm, vias 2 -> 0
- net STAT_LED4: track 426.9 -> 0.00 mm
- net STAT_LED5: track 368.2 -> 0.00 mm
- net STAT_LED6: track 309.7 -> 0.00 mm
- net STAT_LED7: track 258.2 -> 0.00 mm
- net STAT_LED8: track 199.6 -> 0.00 mm
- net STAT_LED9: track 139.1 -> 0.00 mm
- net STAT_LED10: track 80.0 -> 0.00 mm
- net TEMP_10: track 85.9 -> 57.9 mm
- net TEMP_3: track 484.4 -> 465.3 mm
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- added copper zone on B.Cu, net GND_pos_con
- added copper zone on F.Cu, net GND_pos_con
Other:
- board size 50 x 643 mm -> 50 x 643.1 mm
- board text added: "+5V"
- board text added: "BOOT"
- board text added: "CAN1_h"
- board text added: "CAN1_l"
- board text added: "CAN2_h"
- board text added: "CAN2_l"
- board text added: "GND"
- board text added: "Order the flex part with with a thickness 0.11mm Stiffner: Polymide, 0.2mm"
- board text added: "RST"
- board text added: "Stiffener: Polyimide Thickness: 0.20mm"
- board text added: "T1"
- board text added: "T10"
- board text added: "Vcharg"
- board text added: "Vmain"
- board text added: "this side up"
- board text removed: "Bottom"
- board text removed: "Edge"
