File: rapid_tank_level_indicator_hardware/rapid_tank_level_indicator.kicad_sch (KiCad schematic)
At the start: 87 parts, among them J1 Conn_01x04_Pin, J17 TC2050, J2 Conn_02x04_Top_Bottom, J3 Conn_02x04_Top_Bottom, SW1 KMR721NGLFS, SW2 KMR721NGLFS, U1 L7805, U10 MCP9700Ax-ETT, U11 TPD4E1U06, U12 MCP9700Ax-ETT, U13 MCP9700Ax-ETT, U14 MCP9700Ax-ETT, U15 MCP9700Ax-ETT, U16 MCP2562-E-SN, U2 L7805, U3 STM32F105RCTx, U4 MCP9700Ax-ETT, U5 AZ1117-3.3, U6 MCP9700Ax-ETT, U7 MCP9700Ax-ETT, U8 MCP9700Ax-ETT, U9 MCP9700Ax-ETT, Y1 8MHz 12pF

Commit message: add connector and rc-filter
Parts:
- removed C13: 330n, Capacitor_SMD:C_0603_1608Metric, symbol Device:C_Small
- removed C14: 100n, Capacitor_SMD:C_0402_1005Metric, symbol Device:C_Small
- removed D1, D10, D11, D12, D13, D14, D15, D6, D8, D9: red, LED_SMD:LED_0603_1608Metric, symbol Device:LED_Small
- removed D4: RB070MM-30TR, Diode_SMD:D_SOD-123F, symbol Diode:SS34
- removed R10, R11, R26, R30, R32, R4, R5, R6, R7, R9: 1k, Resistor_SMD:R_0402_1005Metric, symbol Device:R_Small
- removed U2: L7805, Package_TO_SOT_SMD:TO-252-2, symbol Regulator_Linear:L7805
- added C13, C14, C18, C19, C22, C23, C26, C27, C28, C30: 1u, Capacitor_SMD:C_0402_1005Metric, symbol Device:C
- added D4: red, LED_SMD:LED_0603_1608Metric, symbol Device:LED_Small
- added J4: Conn_01x12, custom_parts_lib:FFC3B07_pad, symbol Connector_Generic:Conn_01x12
- added J5: FFC3B07-12-T, custom_parts_lib:FFC3B0712T, symbol custom-parts-lib:FFC3B07-12-T
- added R10, R11, R13, R14, R15, R4, R5, R6, R7, R9: 10k, Resistor_SMD:R_0402_1005Metric, symbol Device:R
- added R12: 1k, Resistor_SMD:R_0402_1005Metric, symbol Device:R_Small
- added TP1, TP10, TP2, TP3, TP4, TP5, TP6, TP7, TP8, TP9: TestPoint, TestPoint:TestPoint_Pad_D1.0mm, symbol Connector:TestPoint
- D3: LCSC# C474026 -> C2286; Manufacturer Everlight Elec -> (none); Part# 19-213/RSC-BS2T2B/3T -> (none)
- D5: LCSC (none) -> C2286; LCSC# C474026 -> (none); Manufacturer Everlight Elec -> (none); Part# 19-213/RSC-BS2T2B/3T -> (none)
- R1: value 220 -> 1k5
- R3: value 220 -> 1k; LCSC (none) -> C11702; LCSC# C112291 -> (none); Manufacturer ROHM Semicon -> (none); Part# ESR03EZPJ221 -> (none)
Connections:
- net +3.3V: now also R3.1, R12.1
- net +5V: now also J5.1; no longer U10.1 (V_{DD}), U12.1 (V_{DD}), U13.1 (V_{DD}), U14.1 (V_{DD}), U15.1 (V_{DD}), U4.1 (V_{DD}), U6.1 (V_{DD}), U7.1 (V_{DD}), U8.1 (V_{DD}), U9.1 (V_{DD})
- net GND: now also C13.2, C14.2, C18.2, C19.2, C22.2, C23.2, C26.2, C27.2, C28.2, C30.2, J5.12, J5.MP1, J5.MP2; no longer D5.1 (K), U10.3 (GND), U12.3 (GND), U13.3 (GND), U14.3 (GND), U15.3 (GND), U4.3 (GND), U6.3 (GND), U7.3 (GND), U8.3 (GND), U9.3 (GND)
- net STAT_LED1: now also U3.39 (PC8), D4.1 (K); no longer U3.35 (PB14)
- net STAT_LED2: now also D5.1 (K), U3.40 (PC9); no longer U3.34 (PB13)
- net TEMP_1: now also J4.2 (Pin_2), TP1.1; no longer U3.27 (PB1)
- net TEMP_10: now also J4.11 (Pin_11), TP10.1; no longer U3.8 (PC0)
- net TEMP_2: now also J4.3 (Pin_3), TP3.1; no longer U3.26 (PB0)
- net TEMP_3: now also J4.4 (Pin_4), TP5.1; no longer U3.25 (PC5)
- net TEMP_4: now also J4.5 (Pin_5), TP7.1; no longer U3.24 (PC4)
- net TEMP_5: now also J4.6 (Pin_6), TP9.1; no longer U3.23 (PA7)
- net TEMP_6: now also J4.7 (Pin_7), TP2.1; no longer U3.22 (PA6)
- net TEMP_7: now also J4.8 (Pin_8), TP4.1; no longer U3.21 (PA5)
- net TEMP_8: now also J4.9 (Pin_9), TP6.1; no longer U3.20 (PA4)
- net TEMP_9: now also J4.10 (Pin_10), TP8.1; no longer U3.17 (PA3)
- net at D5.2 (A): now also R12.2; no longer R3.2
- net STAT_LED3: no longer names the net of U3.33 (PB12)
- net STAT_LED4: no longer names the net of U3.30 (PB11)
- net STAT_LED5: no longer names the net of U3.29 (PB10)
- net STAT_LED6: no longer names the net of U3.28 (PB2)
- net STAT_LED7: no longer names the net of U3.10 (PC2)
- net STAT_LED8: no longer names the net of U3.11 (PC3)
- new net: D4.2 (A), R3.2
- new net: C19.1, R7.1, U3.20 (PA4)
- new net: C18.1, R5.1, U3.21 (PA5)
- new net: C22.1, R9.1, U3.17 (PA3)
- new net: C30.1, R15.2, U3.8 (PC0)
- new net: C23.1, R11.1, U3.27 (PB1)
- new net: C27.1, R13.2, U3.24 (PC4)
- new net: C28.1, R14.2, U3.25 (PC5)
- new net: C14.1, R4.1, U3.22 (PA6)
- new net: C13.1, R6.1, U3.23 (PA7)
- new net: C26.1, R10.1, U3.26 (PB0)
- new net +5V_post_con: J4.12 (Pin_12), U10.1 (V_{DD}), U12.1 (V_{DD}), U13.1 (V_{DD}), U14.1 (V_{DD}), U15.1 (V_{DD}), U4.1 (V_{DD}), U6.1 (V_{DD}), U7.1 (V_{DD}), U8.1 (V_{DD}), U9.1 (V_{DD})
- new net GND_pos_con: J4.1 (Pin_1), U10.3 (GND), U12.3 (GND), U13.3 (GND), U14.3 (GND), U15.3 (GND), U4.3 (GND), U6.3 (GND), U7.3 (GND), U8.3 (GND), U9.3 (GND)
- new net TEMP_10_con: J5.2, R15.1
- new net TEMP_1_con: J5.11, R11.2
- new net TEMP_2_con: J5.10, R10.2
- new net TEMP_3_con: J5.9, R14.1
- new net TEMP_4_con: J5.8, R13.1
- new net TEMP_5_con: J5.7, R6.2
- new net TEMP_6_con: J5.6, R4.2
- new net TEMP_7_con: J5.5, R5.2
- new net TEMP_8_con: J5.4, R7.2
- new net TEMP_9_con: J5.3, R9.2
- no-connect marks 24 -> 30
Other:
- note added: "@TODO was für einen Widerstand für die LED?"
- note added: "Connector"
- note added: "General purpose status LEDs"
- note added: "RC filter for 15.9 Hz Cuttoff frequency"
- note removed: "Tank level indicator LEDs"
- moved on the sheet: C15, R2, R8, SW1, SW2
